File: current revision/pwr supply rev 5.kicad_pcb (KiCad board)
At the start: 2 copper layers, 156.6 x 120 mm, 46 parts, among them J1 Conn_WallPlug_Earth, J2 DB9_Female_MountingHoles, P1 R_POT, P2 R_POT, U1 LTM8022

Commit message: initial commit for new layout, smaller board, new AC entry module
Parts:
- added FID1: Fiducial, Fiducial:Fiducial_0.75mm_Mask1.5mm, F.Cu at (2.00, 3.65)
- added FID2: Fiducial, Fiducial:Fiducial_0.75mm_Mask1.5mm, F.Cu at (118.8, 3.65)
- added FID3: Fiducial, Fiducial:Fiducial_0.75mm_Mask1.5mm, F.Cu at (118.5, 96.3)
- added LOGO1: Squid Logo, user_generated_footprints:SquidLogo20x24, F.Cu at (11.4, 84.8)
- C1, C10, C11, C15, C16, C19, C2, C20, C21, C22, C23, C24, C25, C26, C3, C6, C7: footprint Capacitors_SMD:C_0603 -> Capacitor_SMD:C_0603_1608Metric
- C14: footprint Capacitors_SMD:C_0805 -> Capacitor_SMD:C_0805_2012Metric
- C27: value 100n?? -> ??
- D1, D2: value 31v -> 16v
- J1: footprint user:AC_receptacle -> user_generated_footprints:PF0030PC
- J2: footprint Connectors:DB9FC -> user_generated_footprints:DB9FC_w_housing_connection
- P1, P2: value R_POT -> ???
- R1, R2: footprint Resistors_SMD:R_0603 -> Resistor_SMD:R_0603_1608Metric
- moved R1 58.2 mm to (64.5, 55.8), turned to 180 degrees
- moved R2 58.0 mm to (64.5, 57.2), turned to 180 degrees
- moved C5 53.8 mm to (77.7, 11.8), turned to 90 degrees
- moved U1 51.2 mm to (70.7, 52.6), turned to 270 degrees
- moved C2 48.0 mm to (83.7, 70.2), turned to 90 degrees
- moved C19 47.9 mm to (82.2, 70.2), turned to 90 degrees
- moved J2 46.5 mm to (106.9, 44.5)
- moved P1 44.8 mm to (110.5, 70.0)
- moved C14 43.5 mm to (76.5, 51.9), turned to 270 degrees
- moved C4 42.9 mm to (76.8, 89.0), turned to 270 degrees
- moved C1 41.5 mm to (76.3, 57.3), turned to 270 degrees
- moved C9 38.3 mm to (88.5, 11.9), turned to 90 degrees
- moved L1 36.8 mm to (76.7, 75.0), turned to 180 degrees
- moved L2 34.9 mm to (76.8, 24.2), turned to 180 degrees
- moved C27 33.1 mm to (104.0, 60.0), turned to 270 degrees
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Connections:
- net /+24v,A renamed /+15v,A
- net /+24v,B renamed /+15v,B
Routing:
- net Earth: track 860.4 -> 0.00 mm, vias 28 -> 0
- net /3.3v: track 109.7 -> 0.00 mm, vias 3 -> 0
- net /+15v,B: track 107.7 -> 0.00 mm
- net /+0v,B: track 105.6 -> 0.00 mm
- net /+15v,A: track 81.5 -> 0.00 mm, vias 2 -> 0
- net Net-(J1-Pad2): track 67.5 -> 0.00 mm
- net Net-(J1-Pad1): track 67.2 -> 0.00 mm
- net GND: track 64.9 -> 0.00 mm
- net Net-(P2-Pad2): track 37.3 -> 0.00 mm
- net Net-(P1-Pad2): track 37.2 -> 0.00 mm
- net Net-(C1-Pad1): track 36.0 -> 0.00 mm
- net Net-(C19-Pad1): track 33.0 -> 0.00 mm
- net Net-(C20-Pad1): track 28.8 -> 0.00 mm
- net Net-(C22-Pad1): track 25.7 -> 0.00 mm
- net Net-(C21-Pad1): track 23.1 -> 0.00 mm
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- removed copper zone on B.Cu, net /+0v,B
- removed copper zone on F.Cu, net /+0v,B
- removed copper zone on B.Cu, net /3.3v
- removed copper zone on F.Cu, net Earth
- removed copper zone on B.Cu, net GND
- removed copper zone on B.Cu, net Net-(C1-Pad1)
Other:
- board size 156.6 x 120 mm -> 120 x 100.8 mm
- board text added: "End panel with plastic bezel installed"
- board text added: "Mounting Slot"
- board text added: "Squidstat power supply 2021 Mar Admiral Instruments"
- board text removed: "Squidstat power supply 2021 Jan 22 Admiral Instruments"
