File: current revision/pwr supply rev 5.sch (KiCad schematic (older format))
At the start: 46 parts, among them J1 Conn_WallPlug_Earth, J2 DB9_Female_MountingHoles, P1 R_POT, P2 R_POT, U1 LTM8022

Commit message: initial commit for new layout, smaller board, new AC entry module
Parts:
- added FID1, FID2, FID3: Fiducial, Fiducial:Fiducial_0.75mm_Mask1.5mm, symbol Mechanical:Fiducial
- added LOGO1: Squid Logo, user_generated_footprints:SquidLogo20x24, symbol user_generated_parts:DummyBlock
- C1: footprint Capacitors_SMD:C_0603 -> Capacitor_SMD:C_0603_1608Metric; Alternative (none) -> C1608X5R1E225K080AE; MPN (none) -> C1608JB1E225M080AB
- C10, C11, C15, C16, C2, C3, C6, C7: footprint Capacitors_SMD:C_0603 -> Capacitor_SMD:C_0603_1608Metric; Alternative (none) -> CL10A105KB8NNNC, GMK107BJ105KAHT; MPN (none) -> GRT188R61H105ME13D
- C12, C13, C17, C18, C4, C5, C8, C9: MPN (none) -> EEU-FR1V561
- C14: footprint Capacitors_SMD:C_0805 -> Capacitor_SMD:C_0805_2012Metric; MPN (none) -> GRM219R61C226ME15KL
- C19, C20, C21, C22, C23, C24, C25, C26: footprint Capacitors_SMD:C_0603 -> Capacitor_SMD:C_0603_1608Metric; MPN (none) -> '885012206089
- C27: value 100n?? -> ??
- D1, D2: value 31v -> 16v; MPN (none) -> TP1.5KE18A
- J1: footprint user:AC_receptacle -> user_generated_footprints:PF0030PC; symbol conn:Conn_WallPlug_Earth -> Connector:Conn_WallPlug_Earth; MPN (none) -> PF0030/PC
- J2: footprint Connectors:DB9FC -> user_generated_footprints:DB9FC_w_housing_connection; symbol conn:DB9_Female_MountingHoles -> Connector:DB9_Female_MountingHoles; MPN (none) -> ID09S33E4GX00LF
- L1, L2, L3, L4, L5, L6, L7, L8: MPN (none) -> ASPI-6045S-100MT
- P1, P2: value R_POT -> ???
- PS1, PS2: symbol pwr-supply-rev-5-rescue:TPP30-115A-D-user -> user:TPP30-115A-D; MPN (none) -> TPP-30-115A-D
- R1: footprint Resistors_SMD:R_0603 -> Resistor_SMD:R_0603_1608Metric; MPN (none) -> ERA-3AEB4222V
- R2: footprint Resistors_SMD:R_0603 -> Resistor_SMD:R_0603_1608Metric; MPN (none) -> RT0603BRD07154KL
- U1: symbol pwr-supply-rev-5-rescue:LTM8022-pwr-supply-rev-3-rescue-pwr-supply-rev-4-rescue-pwr-supply-rev-4-rescue -> user:LTM8022; MPN (none) -> LTM8022EV#PBF
Connections:
- net +24v,A renamed +15v,A
- net +24v,B renamed +15v,B
